Commit message: Week 6 Rotation still doesnt work

File: src/my_r2d2/urdf/r2d2.urdf.xacro (robot description, xacro)
@@ -220,3 +220,10 @@
     <origin xyz="0 0 ${(bodylen/2)+wheeldiam+0.1}"/>
   </joint>
+  <link name="eye">
+  </link>
+  <joint name="toeye" type="fixed">
+    <parent link="box"/>
+    <child link="eye"/>
+    <origin xyz="0 0 0"  rpy="${-pi/2} 0 ${-pi/2}"/>
+  </joint>
 </robot>
